Commit message: add arm2 urdf

File: src/arm_desciption/urdf/Part1.urdf (robot description, URDF)
Before this commit: robot arm, 1 links, 0 joints
Links:
- removed link arm
- added link Part1, mass 0.31856; collision mesh filename=package://arm_desciption/meshes/Part1.STL; visual mesh filename=package://arm_desciption/meshes/Part1.STL
